File: Hardware/TAS5806M_Breakout_Hardware/TAS5806M_Breakout_Hardware.kicad_pcb (KiCad board)
At the start: 2 copper layers, 63.5 x 50.8 mm, 32 parts, among them J1 Headers, J2 Power Input, U1 TAS5806M

Commit message: Finalized design, generated Gerbs
Parts:
- added C21: 10uF, Capacitor_SMD:C_0603_1608Metric_Pad1.05x0.95mm_HandSolder, F.Cu at (165.7, 77.3)
- added C22: 10uF, Capacitor_SMD:C_0603_1608Metric_Pad1.05x0.95mm_HandSolder, F.Cu at (165.7, 79.2)
- added G***: LOGO, ESP8266:Signature, F.Cu at (184.2, 121.4)
- added G***: LOGO, ESP8266:lizard_logo, F.Cu at (148.1, 114.6)
- added U2: OKI, MRDT_Devices:OKI_Horizontal, F.Cu at (162.0, 76.5)
- C3, C5: footprint Capacitor_SMD:C_0603_1608Metric_Pad1.05x0.95mm_HandSolder -> Capacitor_SMD:C_1206_3216Metric_Pad1.42x1.75mm_HandSolder
- moved C1 3.24 mm to (147.5, 87.8), turned to 90 degrees
- moved C5 0.62 mm to (154.4, 87.8)
- moved C3 0.60 mm to (154.4, 109.0)
- moved C15 0.29 mm to (178.2, 91.0)
- moved C19 0.29 mm to (175.3, 91.0)
- moved C13 0.25 mm to (178.2, 86.8)
- moved C17 0.25 mm to (175.3, 86.8)
- moved C2 0.19 mm to (150.1, 87.8), turned to 90 degrees
Connections:
- J2 pad 1: GND -> +12V
- J2 pad 2: +12V -> GND
Routing:
- net +3V3: track 49.3 -> 82.2 mm
- net +12V: track 126.3 -> 142.7 mm
- net Net-(C15-Pad1): track 0.00 -> 6.17 mm
- net Net-(C13-Pad1): track 0.00 -> 5.97 mm
- net GND: track 18.0 -> 20.8 mm, vias 13 -> 93
- net (no net): vias 0 -> 5
- added copper zone on F.Cu, net Net-(C13-Pad1)
- added copper zone on F.Cu, net Net-(C15-Pad1)
Other:
- outline, holes or cut-outs redrawn
- board text added: "+"
- board text added: "-"
- board text added: "3v3"
- board text added: "ADR/F"
- board text added: "Audio Amplifier Breakout Board Rev 1, 2020 Dan Napierkowski"
- board text added: "GND"
- board text added: "LRCLK"
- board text added: "Left Channel Speaker"
- board text added: "PDN"
- board text added: "Right Channel Speaker"
- board text added: "SCL"
- board text added: "SCLK"
- board text added: "SDA"
- board text added: "SDIN"
- board text added: "SDOUT"
- board text added: "Vin"
