File: Hardware/TAS5806M_Breakout_Hardware/_autosave-TAS5806M_Breakout_Hardware.sch (KiCad schematic (older format))
At the start: 35 parts, among them J1 Headers, J2 Power Input, U1 TAS5806M, U2 OKI

Commit message: Finalized design, generated Gerbs
Parts:
- C3, C5: footprint Capacitor_SMD:C_0603_1608Metric_Pad1.05x0.95mm_HandSolder -> Capacitor_SMD:C_1206_3216Metric_Pad1.42x1.75mm_HandSolder
Changed lines of the file:
@@
 F 0 "C5" H 3750 2800 50  0000 C CNN
 F 1 "22uF" H 3800 2700 50  0000 C CNN
-F 2 "Capacitor_SMD:C_0603_1608Metric_Pad1.05x0.95mm_HandSolder" H 3638 2600 50  0001 C CNN
+F 2 "Capacitor_SMD:C_1206_3216Metric_Pad1.42x1.75mm_HandSolder" H 3638 2600 50  0001 C CNN
 F 3 "~" H 3600 2750 50  0001 C CNN
 	1    3600 2750
@@
 F 0 "C3" H 2700 3050 50  0000 C CNN
 F 1 "22uF" H 2750 2950 50  0000 C CNN
-F 2 "Capacitor_SMD:C_0603_1608Metric_Pad1.05x0.95mm_HandSolder" H 2588 2850 50  0001 C CNN
+F 2 "Capacitor_SMD:C_1206_3216Metric_Pad1.42x1.75mm_HandSolder" H 2588 2850 50  0001 C CNN
 F 3 "~" H 2550 3000 50  0001 C CNN
 	1    2550 3000
